File: PCB/starbie.kicad_pcb (KiCad board)
At the start: 2 copper layers, 62 x 50.5 mm, 7 parts, among them J1 Conn_01x04_Pin, J2 Conn_01x08_Pin, SW1 SW_Push, SW2 SW_Push, U1 XIAO-ESP32-C3-SMD, U2 DHT11

Commit message: Added README, BOM, 3D renders; Flipped Motion Sensor orientation in PCB
Parts:
- moved J2 17.4 mm to (104.0, 88.3), turned to 0 degrees
Routing:
- net +3.3V: track 53.0 -> 42.5 mm
- net /SCL: track 29.8 -> 23.6 mm
- net /GPIO2: track 42.8 -> 41.3 mm, vias 0 -> 1
